File: PCB/STM32L4_Project/STM32L4_Project.kicad_sch (KiCad schematic)
At the start: 37 parts, among them J1 USB_B_Micro, J2 Conn_01x07_Male, J3 Conn_01x03_Female, J4 ARM 10pin, U1 XC6206P332MR, U2 LM386, U3 USBLC6-2SC6, U4 STM32L432KBU6

Commit message: More work on PCB
Parts:
- removed C12: 100n, Capacitor_SMD:C_0402_1005Metric, symbol Device:C
- removed C6: 100u, Capacitor_SMD:C_0805_2012Metric, symbol Device:C
- added H1, H2, H3, H4: MountingHole, MountingHole:MountingHole_2.2mm_M2, symbol Mechanical:MountingHole
- C5: value 0.1u -> 10pF
- J1: footprint Connector_USB:USB_Micro-B_Wuerth_629105150521 -> Connector_USB:USB_Micro-B_Molex_47346-0001
- R1: value 10k -> 100
- renumbered C11 to C10, C13 to C11, C14 to C12, C15 to C13, C16 to C14, C7 to C6, C8 to C7, C9 to C8, C10 to C9
Connections:
- net +5V: now also J2.7 (Pin_7); no longer J2.5 (Pin_5)
- net ADC_IN: now also C5.2, U2.5
- net GND: now also J2.5 (Pin_5); no longer J2.7 (Pin_7)
- net PA3: now also J2.3 (Pin_3); no longer J2.1 (Pin_1)
- net PA8: now also J2.1 (Pin_1); no longer J2.3 (Pin_3)
Other:
- note added: "Mounting Holes"
