File: PCB/PCB_v2/PCB_v2.kicad_sch (KiCad schematic)
At the start: 17 parts, among them U1 ADAU1979xBCP

Commit message: Collected more human walking data in radar lab
Other:
- note added: "Device configured in I2C mode"
Changed lines of the file:
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@@
+		)
+	)
+	(text "Device configured in I2C mode\n"
+		(exclude_from_sim no)
+		(at 252.984 55.118 0)
+		(effects
+			(font
+				(size 0.635 0.635)
+			)
 		)
 	)
